Commit message: modified:   src/omnicar/description/robot.urdf.xacro 	modified:   src/omnicar/description/ros2_control.xacro 	modified:   src/omnicar/launch/launch_bot.launch.py 	modified:   src/omnicar/launch/launch_sim.launch.py 	modified:   src/omnicar/launch/rsp.launch.py

File: src/omnicar/description/robot.urdf.xacro (robot description, xacro)
@@ -1,4 +1,5 @@
 <?xml version="1.0"?>
 <robot xmlns:xacro="http://www.ros.org/wiki/xacro"  name="robot">
+  <xacro:arg name='sim_mode' default='true'/>
     <xacro:include filename="robot_core.xacro" />
     <xacro:include filename="ros2_control.xacro" />

File: src/omnicar/description/ros2_control.xacro (robot description, xacro)
@@ -1,90 +1,100 @@
 <?xml version="1.0"?>
 <robot xmlns:xacro="http://www.ros.org/wiki/xacro">
-  <!-- <ros2_control name="GazeboSystem" type="system">
-    <hardware>
-        <plugin>gazebo_ros2_control/GazeboSystem</plugin>
-    </hardware>
-    <joint name="rear_right_wheel_joint">
-        <command_interface name="velocity">
-            <param name="min">-10</param>
-            <param name="max">10</param>
-        </command_interface>
-        <state_interface name="position" />
-        <state_interface name="velocity" />
-    </joint>
-    <joint name="rear_left_wheel_joint">
-        <command_interface name="velocity">
-            <param name="min">-10</param>
-            <param name="max">10</param>
-        </command_interface>
-        <state_interface name="velocity" />
-        <state_interface name="position" />
-    </joint>
-     <joint name="front_right_wheel_joint">
-        <command_interface name="velocity">
-            <param name="min">-10</param>
-            <param name="max">10</param>
-        </command_interface>
-        <state_interface name="position" />
-        <state_interface name="velocity" />
-    </joint>
-    <joint name="front_left_wheel_joint">
-        <command_interface name="velocity">
-            <param name="min">-10</param>
-            <param name="max">10</param>
-        </command_interface>
-        <state_interface name="velocity" />
-        <state_interface name="position" />
-    </joint>
-  </ros2_control> -->
-<ros2_control name="RealBot" type="system">
-    <hardware>
-        <plugin>arduino_hardware_controller/ArduinoHardwareController</plugin>
-        <param name="front_left_wheel_name">front_left_wheel_joint</param>
-        <param name="front_right_wheel_name">front_right_wheel_joint</param>
-        <param name="back_left_wheel_name">rear_left_wheel_joint</param>
-        <param name="back_right_wheel_name">rear_right_wheel_joint</param>
-        <param name="loop_rate">30.00</param>
-        <param name="device">/dev/ttyUSB0</param>
-        <param name="baud_rate">9600</param>
-        <param name="timeout">1000</param>
+  <xacro:unless value="$(arg sim_mode)">
+    <ros2_control name="GazeboSystem" type="system">
+      <hardware>
+          <plugin>gazebo_ros2_control/GazeboSystem</plugin>
       </hardware>
-    <joint name="rear_right_wheel_joint">
-        <command_interface name="velocity">
-            <param name="min">-10</param>
-            <param name="max">10</param>
-        </command_interface>
-        <state_interface name="position" />
-        <state_interface name="velocity" />
-    </joint>
-    <joint name="rear_left_wheel_joint">
-        <command_interface name="velocity">
-            <param name="min">-10</param>
-            <param name="max">10</param>
-        </command_interface>
-        <state_interface name="velocity" />
-        <state_interface name="position" />
-    </joint>
-     <joint name="front_right_wheel_joint">
-        <command_interface name="velocity">
-            <param name="min">-10</param>
-            <param name="max">10</param>
-        </command_interface>
-        <state_interface name="position" />
-        <state_interface name="velocity" />
-    </joint>
-    <joint name="front_left_wheel_joint">
-        <command_interface name="velocity">
-            <param name="min">-10</param>
-            <param name="max">10</param>
-        </command_interface>
-        <state_interface name="velocity" />
-        <state_interface name="position" />
-    </joint>
-  </ros2_control>
-  <gazebo>
+      <joint name="rear_right_wheel_joint">
+          <command_interface name="velocity">
+              <param name="min">-10</param>
+              <param name="max">10</param>
+          </command_interface>
+          <state_interface name="position" />
+          <state_interface name="velocity" />
+      </joint>
+      <joint name="rear_left_wheel_joint">
+          <command_interface name="velocity">
+              <param name="min">-10</param>
+              <param name="max">10</param>
+          </command_interface>
+          <state_interface name="velocity" />
+          <state_interface name="position" />
+      </joint>
+      <joint name="front_right_wheel_joint">
+          <command_interface name="velocity">
+              <param name="min">-10</param>
+              <param name="max">10</param>
+          </command_interface>
+          <state_interface name="position" />
+          <state_interface name="velocity" />
+      </joint>
+      <joint name="front_left_wheel_joint">
+          <command_interface name="velocity">
+              <param name="min">-10</param>
+              <param name="max">10</param>
+          </command_interface>
+          <state_interface name="velocity" />
+          <state_interface name="position" />
+      </joint>
+    </ros2_control>
+    <gazebo>
       <plugin name="gazebo_ros2_control" filename="libgazebo_ros2_control.so">
         <parameters>$(find omnicar)/config/my_controllers.yaml</parameters>
+        <parameters>$(find omnicar)/config/sim.yaml</parameters>
       </plugin>
-  </gazebo>
+    </gazebo>
+  </xacro:unless>
+  <xacro:if value="$(arg sim_mode)">
+    <ros2_control name="RealBot" type="system">
+      <hardware>
+          <plugin>arduino_hardware_controller/ArduinoHardwareController</plugin>
+          <param name="front_left_wheel_name">front_left_wheel_joint</param>
+          <param name="front_right_wheel_name">front_right_wheel_joint</param>
+          <param name="back_left_wheel_name">rear_left_wheel_joint</param>
+          <param name="back_right_wheel_name">rear_right_wheel_joint</param>
+          <param name="loop_rate">30.00</param>
+          <param name="device">/dev/ttyUSB0</param>
+          <param name="baud_rate">9600</param>
+          <param name="timeout">1000</param>
+        </hardware>
+      <joint name="rear_right_wheel_joint">
+          <command_interface name="velocity">
+              <param name="min">-10</param>
+              <param name="max">10</param>
+          </command_interface>
+          <state_interface name="position" />
+          <state_interface name="velocity" />
+      </joint>
+      <joint name="rear_left_wheel_joint">
+          <command_interface name="velocity">
+              <param name="min">-10</param>
+              <param name="max">10</param>
+          </command_interface>
+          <state_interface name="velocity" />
+          <state_interface name="position" />
+      </joint>
+      <joint name="front_right_wheel_joint">
+          <command_interface name="velocity">
+              <param name="min">-10</param>
+              <param name="max">10</param>
+          </command_interface>
+          <state_interface name="position" />
+          <state_interface name="velocity" />
+      </joint>
+      <joint name="front_left_wheel_joint">
+          <command_interface name="velocity">
+              <param name="min">-10</param>
+              <param name="max">10</param>
+          </command_interface>
+          <state_interface name="velocity" />
+          <state_interface name="position" />
+      </joint>
+    </ros2_control>
+    <gazebo>
+        <plugin name="gazebo_ros2_control" filename="libgazebo_ros2_control.so">
+          <parameters>$(find omnicar)/config/my_controllers.yaml</parameters>
+        </plugin>
+    </gazebo>
+  </xacro:if>
 </robot>
