Commit message: Fixed IMU Sensor

File: src/omnicar/description/imu.xacro (robot description, xacro)
@@ -11,16 +11,17 @@
         <box size="0.010 0.03 0.03"/>
       </geometry>
-      <material name="red"/>
     </visual>
   </link>
   <gazebo reference="gyro_link">
-    <material>Gazebo/Red</material>
-    <sensor name="imu_sensor" type="imu">
-      <always_on>1</always_on>
-      <update_rate>1</update_rate>
-      <visualize>true</visualize>
-      <topic>imu</topic>
-      <plugin filename="gz-sim-imu-system"
-        name="gz::sim::systems::Imu">
+    <sensor name="imu_link" type="imu">
+      <!-- ensure the sensor is active (required) -->
+      <always_on>true</always_on>
+      <update_rate>30</update_rate>
+      <plugin name="imu_plugin" filename="libgazebo_ros_imu_sensor.so">
+        <ros>
+          <!-- publish to /imu/data -->
+          <namespace>/imu</namespace>
+          <remapping>~/out:=/imu</remapping>
+        </ros>
       </plugin>
     </sensor>
