Commit message: added camera to sim and realbot

File: src/omnicar/description/camera.xacro (robot description, xacro)
@@ -2,5 +2,5 @@
 <robot xmlns:xacro="http://www.ros.org/wiki/xacro">
   <joint name="camera_joint" type="fixed">
-    <parent link="chassis"/>
+    <parent link="base_link"/>
     <child link="camera_link"/>
     <origin xyz="0.305 0 0.08" rpy="0 0 0"/>
@@ -15,5 +15,4 @@
   </link>
   <gazebo reference="camera_link">
-    <material>Gazebo/Red</material>
     <sensor name="camera" type="camera">
       <pose> 0 0 0 0 0 0 </pose>

File: src/omnicar/description/robot.urdf.xacro (robot description, xacro)
@@ -7,4 +7,4 @@
     <xacro:include filename="imu.xacro" />
     <xacro:include filename="gps.xacro" />
-    <!-- <xacro:include filename="camera.xacro" /> add camera -->
+    <xacro:include filename="camera.xacro" /> add camera
 </robot>

Commit message: removed red from camera link

File: src/omnicar/description/camera.xacro (robot description, xacro)
@@ -11,5 +11,4 @@
         <box size="0.010 0.03 0.03"/>
       </geometry>
-      <material name="red"/>
     </visual>
   </link>

Commit message: xacro file updates (fixed foxglove viewing)

File: src/omnicar/description/camera.xacro (robot description, xacro)
@@ -2,5 +2,5 @@
 <robot xmlns:xacro="http://www.ros.org/wiki/xacro">
   <joint name="camera_joint" type="fixed">
-    <parent link="base_link"/>
+    <parent link="chassis"/>
     <child link="camera_link"/>
     <origin xyz="0.305 0 0.08" rpy="0 0 0"/>

File: src/omnicar/description/gps.xacro (robot description, xacro)
@@ -2,5 +2,5 @@
 <robot xmlns:xacro="http://www.ros.org/wiki/xacro">
   <joint name="gps_joint" type="fixed">
-    <parent link="base_link"/>
+    <parent link="chassis"/>
     <child link="gps_link"/>
     <origin xyz="0.305 0 0.08" rpy="0 0 0"/>

File: src/omnicar/description/imu.xacro (robot description, xacro)
@@ -2,5 +2,5 @@
 <robot xmlns:xacro="http://www.ros.org/wiki/xacro">
   <joint name="gyro_joint" type="fixed">
-    <parent link="base_link"/>
+    <parent link="chassis"/>
     <child link="gyro_link"/>
     <origin xyz="0.305 0 0.08" rpy="0 0 0"/>

File: src/omnicar/description/robot_core.xacro (robot description, xacro)
@@ -3,4 +3,6 @@
   <xacro:include filename="$(find omnicar)/description/urdf/mecanum_wheel_macro.xacro" />
   <link name="base_link">
+  </link>
+  <link name="chassis">
     <visual>
       <geometry>
@@ -21,5 +23,5 @@
     </inertial>
   </link>
-  <gazebo reference="base_link">
+  <gazebo reference="chassis">
     <mu1 value="0.6"/>
     <mu2 value="0.6"/>
@@ -28,4 +30,9 @@
     <fdir1 value="0 1 0"/>
   </gazebo>
+  <joint name="chassis" type="fixed">
+    <origin xyz="0 0 0.2" rpy="0 0 0" />
+    <parent link="base_link" />
+    <child link="chassis" />
+  </joint>
   <xacro:mecanum_wheel name="front_right" side="1"  interface="hardware_interface/EffortJointInterface"/>
   <xacro:mecanum_wheel name="front_left"  side="-1" interface="hardware_interface/EffortJointInterface"/>
@@ -35,5 +42,5 @@
     <origin xyz="0.3 -0.25 -0.1" rpy="0 0 ${pi/2}" />
     <axis xyz="1 0 0" />
-    <parent link="base_link" />
+    <parent link="chassis" />
     <child link="front_right_wheel_link" />
   </joint>
@@ -41,5 +48,5 @@
     <origin xyz="0.3 0.25 -0.1" rpy="0 0 ${pi/2}" />
     <axis xyz="1 0 0" />
-    <parent link="base_link" />
+    <parent link="chassis" />
     <child link="front_left_wheel_link" />
   </joint>
@@ -47,5 +54,5 @@
     <origin xyz="-0.3 -0.25 -0.1" rpy="0 0 ${pi/2}" />
     <axis xyz="1 0 0" />
-    <parent link="base_link" />
+    <parent link="chassis" />
     <child link="rear_right_wheel_link" />
   </joint>
@@ -53,5 +60,5 @@
     <origin xyz="-0.3 0.25 -0.1" rpy="0 0 ${pi/2}" />
     <axis xyz="1 0 0" />
-    <parent link="base_link" />
+    <parent link="chassis" />
     <child link="rear_left_wheel_link" />
   </joint>

File: src/omnicar/description/urdf/rollers.xacro (robot description, xacro)
@@ -15,10 +15,20 @@
           <origin xyz="0 0 0" rpy="0 0 0" />
           <geometry>
-            <mesh filename="$(find omnicar)/description/mesh/visual/roller.dae" scale="1 1 1" />
+            <xacro:if value="$(arg sim_mode)">
+              <mesh filename="$(find omnicar)/description/mesh/visual/roller.dae" scale="1 1 1" />
+            </xacro:if>
+            <xacro:unless value="$(arg sim_mode)">
+              <mesh filename="package://omnicar/description/mesh/visual/roller.dae" scale="1 1 1" />
+            </xacro:unless>
           </geometry>
         </visual>
         <collision>
           <geometry>
-            <mesh filename="$(find omnicar)/description/mesh/collision/roller.stl" scale="1 1 1" />
+            <xacro:if value="$(arg sim_mode)">
+              <mesh filename="$(find omnicar)/description/mesh/visual/roller.dae" scale="1 1 1" />
+            </xacro:if>
+            <xacro:unless value="$(arg sim_mode)">
+              <mesh filename="package://omnicar/description/mesh/visual/roller.dae" scale="1 1 1" />
+            </xacro:unless>
           </geometry>
         </collision>

File: src/omnicar/description/urdf/wheel.xacro (robot description, xacro)
@@ -6,10 +6,20 @@
         <origin xyz="0 0 0" rpy="0 0 0" />
         <geometry>
-          <mesh filename="$(find omnicar)/description/mesh/visual/wheel.dae" scale="${side} 1 1" />
+          <xacro:if value="$(arg sim_mode)">
+            <mesh filename="$(find omnicar)/description/mesh/visual/wheel.dae" scale="${side} 1 1" />
+          </xacro:if>
+          <xacro:unless value="$(arg sim_mode)">
+            <mesh filename="package://omnicar/description/mesh/visual/wheel.dae" scale="${side} 1 1" />
+          </xacro:unless>
         </geometry>
       </visual>
       <collision>
         <geometry>
-          <mesh filename="$(find omnicar)/description/mesh/collision/wheel.stl" scale="${side} 1 1" />
+          <xacro:if value="$(arg sim_mode)">
+            <mesh filename="$(find omnicar)/description/mesh/visual/wheel.dae" scale="${side} 1 1" />
+          </xacro:if>
+          <xacro:unless value="$(arg sim_mode)">
+            <mesh filename="package://omnicar/description/mesh/visual/wheel.dae" scale="${side} 1 1" />
+          </xacro:unless>
         </geometry>
       </collision>
