Commit message: 2/04/25 robot

File: src/example_2/description/urdf/diffbot.urdf.xacro (robot description, xacro)
@@ -8,4 +8,7 @@
   <xacro:include filename="$(find ros2_control_demo_description)/diffbot/urdf/diffbot.materials.xacro" />
   <!-- Import diffbot ros2_control description -->
-  <xacro:include filename="$(find arduino_hardware_controller)/ros2_control/diffbot.ros2_control.xacro" />
+  <xacro:include filename="$(find ros2_control_demo_example_2)/ros2_control/diffbot.ros2_control.xacro" />
+  <xacro:diffbot prefix="$(arg prefix)" />
+  <xacro:diffbot_ros2_control
+    name="DiffBot" prefix="$(arg prefix)" use_mock_hardware="$(arg use_mock_hardware)"/>
 </robot>

File: src/omnicar/description/ros2_control.xacro (robot description, xacro)
@@ -49,5 +49,5 @@
     <ros2_control name="RealBot" type="system">
       <hardware>
-          <plugin>arduino_hardware_controller/ArduinoSysHardware</plugin>
+          <plugin>ros2_control_demo_example_2/DiffBotSystemHardware</plugin>
           <param name="front_left_wheel_name">front_left_wheel_joint</param>
           <param name="front_right_wheel_name">front_right_wheel_joint</param>
@@ -92,4 +92,33 @@
       </joint>
     </ros2_control>
+<!-- <ros2_control name="RealRobot" type="system">
+      <hardware>
+          <plugin>diffdrive_arduino/DiffDriveArduino</plugin>
+          <param name="left_wheel_name">back_left_wheel_joint</param>
+          <param name="right_wheel_name">back_right_wheel_joint</param>
+          <param name="loop_rate">30</param>
+          <param name="device">/dev/ttyUSB0</param>
+          <param name="baud_rate">57600</param>
+          <param name="timeout">1000</param>
+          <param name="enc_counts_per_rev">3436</param>
+      </hardware>
+      Note everything below here is the same as the Gazebo one
+      <joint name="back_left_wheel_joint">
+          <command_interface name="velocity">
+              <param name="min">-10</param>
+              <param name="max">10</param>
+          </command_interface>
+          <state_interface name="velocity"/>
+          <state_interface name="position"/>
+      </joint>
+      <joint name="back_right_wheel_joint">
+          <command_interface name="velocity">
+              <param name="min">-10</param>
+              <param name="max">10</param>
+          </command_interface>
+          <state_interface name="velocity"/>
+          <state_interface name="position"/>
+      </joint>
+    </ros2_control> -->
     <gazebo>
         <plugin name="gazebo_ros2_control" filename="libgazebo_ros2_control.so">
