Commit message: latest robot

File: install/omnicar/share/omnicar/description/camera.xacro (robot description, xacro)
@@ -1,45 +1 @@
-<?xml version="1.0"?>
-<robot xmlns:xacro="http://www.ros.org/wiki/xacro">
-  <joint name="camera_joint" type="fixed">
-    <parent link="chassis"/>
-    <child link="camera_link"/>
-    <origin xyz="0.305 0 0.08" rpy="0 0 0"/>
-  </joint>
-  <link name="camera_link">
-    <visual>
-      <geometry>
-        <box size="0.010 0.03 0.03"/>
-      </geometry>
-      <material name="red"/>
-    </visual>
-  </link>
-  <gazebo reference="camera_link">
-    <material>Gazebo/Red</material>
-    <sensor name="camera" type="camera">
-      <pose> 0 0 0 0 0 0 </pose>
-      <visualize>true</visualize>
-      <update_rate>10</update_rate>
-      <camera>
-        <horizontal_fov>1.089</horizontal_fov>
-        <image>
-          <format>R8G8B8</format>
-          <width>640</width>
-          <height>480</height>
-        </image>
-        <clip>
-          <near>0.05</near>
-          <far>8.0</far>
-        </clip>
-      </camera>
-      <plugin name="camera_controller" filename="libgazebo_ros_camera.so">
-        <frame_name>camera_link_optical</frame_name>
-      </plugin>
-    </sensor>
-  </gazebo>
-  <joint name="camera_optical_joint" type="fixed">
-    <origin xyz="0 0 0" rpy="${-pi/2} 0 ${-pi/2}" />
-    <parent link="camera_link" />
-    <child link="camera_link_optical" />
-  </joint>
-  <link name="camera_link_optical"></link>
-</robot>
+/home/nwhit210/omnicar_ws/src/omnicar/description/camera.xacro

File: install/omnicar/share/omnicar/description/robot.urdf.xacro (robot description, xacro)
@@ -1,7 +1 @@
-<?xml version="1.0"?>
-<robot xmlns:xacro="http://www.ros.org/wiki/xacro"  name="robot">
-  <xacro:arg name='sim_mode' default='true'/>
-    <xacro:include filename="robot_core.xacro" />
-    <xacro:include filename="ros2_control.xacro" />
-    <!-- <xacro:include filename="camera.xacro" /> add camera -->
-</robot>
+/home/nwhit210/omnicar_ws/src/omnicar/description/robot.urdf.xacro

File: install/omnicar/share/omnicar/description/robot_core.xacro (robot description, xacro)
@@ -1,58 +1 @@
-<?xml version="1.0" ?>
-<robot name="mecanum_wheel_robot" xmlns:xacro="http://ros.org/wiki/xacro">
-  <xacro:include filename="$(find omnicar)/description/urdf/mecanum_wheel_macro.xacro" />
-  <link name="base_link">
-    <visual>
-      <geometry>
-        <box size="0.7 0.4 0.3" />
-      </geometry>
-    </visual>
-    <collision>
-      <geometry>
-        <box size="0.7 0.4 0.3" />
-      </geometry>
-    </collision>
-    <inertial>
-      <origin xyz="0 0 0" />
-      <mass value="10.0" />
-      <inertia ixx="0.83333" ixy="0.0" ixz="0.0"
-              iyy="1.9333" iyz="0.0"
-              izz="2.1667" />
-    </inertial>
-  </link>
-  <gazebo reference="base_link">
-    <mu1 value="0.6"/>
-    <mu2 value="0.6"/>
-    <kp value="10000000.0" />
-    <kd value="1.0" />
-    <fdir1 value="0 1 0"/>
-  </gazebo>
-  <xacro:mecanum_wheel name="front_right" side="1"  interface="hardware_interface/EffortJointInterface"/>
-  <xacro:mecanum_wheel name="front_left"  side="-1" interface="hardware_interface/EffortJointInterface"/>
-  <xacro:mecanum_wheel name="rear_right"  side="-1" interface="hardware_interface/EffortJointInterface"/>
-  <xacro:mecanum_wheel name="rear_left"   side="1"  interface="hardware_interface/EffortJointInterface"/>
-  <joint name="front_right_wheel_joint" type="continuous">
-    <origin xyz="0.3 -0.25 -0.1" rpy="0 0 ${pi/2}" />
-    <axis xyz="1 0 0" />
-    <parent link="base_link" />
-    <child link="front_right_wheel_link" />
-  </joint>
-  <joint name="front_left_wheel_joint" type="continuous">
-    <origin xyz="0.3 0.25 -0.1" rpy="0 0 ${pi/2}" />
-    <axis xyz="1 0 0" />
-    <parent link="base_link" />
-    <child link="front_left_wheel_link" />
-  </joint>
-  <joint name="rear_right_wheel_joint" type="continuous">
-    <origin xyz="-0.3 -0.25 -0.1" rpy="0 0 ${pi/2}" />
-    <axis xyz="1 0 0" />
-    <parent link="base_link" />
-    <child link="rear_right_wheel_link" />
-  </joint>
-  <joint name="rear_left_wheel_joint" type="continuous">
-    <origin xyz="-0.3 0.25 -0.1" rpy="0 0 ${pi/2}" />
-    <axis xyz="1 0 0" />
-    <parent link="base_link" />
-    <child link="rear_left_wheel_link" />
-  </joint>
-</robot>
+/home/nwhit210/omnicar_ws/src/omnicar/description/robot_core.xacro

File: install/omnicar/share/omnicar/description/ros2_control.xacro (robot description, xacro)
@@ -1,100 +1 @@
-<?xml version="1.0"?>
-<robot xmlns:xacro="http://www.ros.org/wiki/xacro">
-  <xacro:if value="$(arg sim_mode)">
-    <ros2_control name="GazeboSystem" type="system">
-      <hardware>
-          <plugin>gazebo_ros2_control/GazeboSystem</plugin>
-      </hardware>
-      <joint name="rear_right_wheel_joint">
-          <command_interface name="velocity">
-              <param name="min">-10</param>
-              <param name="max">10</param>
-          </command_interface>
-          <state_interface name="position" />
-          <state_interface name="velocity" />
-      </joint>
-      <joint name="rear_left_wheel_joint">
-          <command_interface name="velocity">
-              <param name="min">-10</param>
-              <param name="max">10</param>
-          </command_interface>
-          <state_interface name="velocity" />
-          <state_interface name="position" />
-      </joint>
-      <joint name="front_right_wheel_joint">
-          <command_interface name="velocity">
-              <param name="min">-10</param>
-              <param name="max">10</param>
-          </command_interface>
-          <state_interface name="position" />
-          <state_interface name="velocity" />
-      </joint>
-      <joint name="front_left_wheel_joint">
-          <command_interface name="velocity">
-              <param name="min">-10</param>
-              <param name="max">10</param>
-          </command_interface>
-          <state_interface name="velocity" />
-          <state_interface name="position" />
-      </joint>
-    </ros2_control>
-    <gazebo>
-      <plugin name="gazebo_ros2_control" filename="libgazebo_ros2_control.so">
-        <parameters>$(find omnicar)/config/my_controllers.yaml</parameters>
-        <parameters>$(find omnicar)/config/sim.yaml</parameters>
-      </plugin>
-    </gazebo>
-  </xacro:if>
-  <xacro:unless value="$(arg sim_mode)">
-    <ros2_control name="RealBot" type="system">
-      <hardware>
-          <plugin>arduino_hardware_controller/ArduinoSysHardware</plugin>
-          <param name="front_left_wheel_name">front_left_wheel_joint</param>
-          <param name="front_right_wheel_name">front_right_wheel_joint</param>
-          <param name="back_left_wheel_name">rear_left_wheel_joint</param>
-          <param name="back_right_wheel_name">rear_right_wheel_joint</param>
-          <param name="loop_rate">30.00</param>
-          <param name="device">/dev/ttyUSB0</param>
-          <param name="baud_rate">9600</param>
-          <param name="timeout_ms">1000</param>
-        </hardware>
-      <joint name="rear_right_wheel_joint">
-          <command_interface name="velocity">
-              <param name="min">-10</param>
-              <param name="max">10</param>
-          </command_interface>
-          <state_interface name="position" />
-          <state_interface name="velocity" />
-      </joint>
-      <joint name="rear_left_wheel_joint">
-          <command_interface name="velocity">
-              <param name="min">-10</param>
-              <param name="max">10</param>
-          </command_interface>
-          <state_interface name="velocity" />
-          <state_interface name="position" />
-      </joint>
-      <joint name="front_right_wheel_joint">
-          <command_interface name="velocity">
-              <param name="min">-10</param>
-              <param name="max">10</param>
-          </command_interface>
-          <state_interface name="position" />
-          <state_interface name="velocity" />
-      </joint>
-      <joint name="front_left_wheel_joint">
-          <command_interface name="velocity">
-              <param name="min">-10</param>
-              <param name="max">10</param>
-          </command_interface>
-          <state_interface name="velocity" />
-          <state_interface name="position" />
-      </joint>
-    </ros2_control>
-    <gazebo>
-        <plugin name="gazebo_ros2_control" filename="libgazebo_ros2_control.so">
-          <parameters>$(find omnicar)/config/my_controllers.yaml</parameters>
-        </plugin>
-    </gazebo>
-  </xacro:unless>
-</robot>
+/home/nwhit210/omnicar_ws/src/omnicar/description/ros2_control.xacro

File: install/omnicar/share/omnicar/description/urdf/mecanum_wheel.urdf.xacro (robot description, xacro)
@@ -1,19 +1 @@
-<?xml version="1.0" ?>
-<robot name="mecanum_wheel_robot" xmlns:xacro="http://ros.org/wiki/xacro">
-  <xacro:include filename="$(find omnicar)/description/urdf/mecanum_wheel_macro.xacro" />
-  <xacro:mecanum_wheel name="front_right" side="1" interface="hardware_interface/EffortJointInterface" />
-  <xacro:mecanum_wheel name="front_left" side="-1" interface="hardware_interface/EffortJointInterface" />
-  <link name="map">
-    <origin xyz="0 0 0" rpy="0 0 0" />
-  </link>
-  <joint name="virtual_map_right" type="fixed">
-    <origin xyz="0.1 0.2 0" />
-    <parent link="map" />
-    <child link="front_right_wheel_link" />
-  </joint>
-  <joint name="virtual_map_left" type="fixed">
-    <origin xyz="-0.1 0.2 0" />
-    <parent link="map" />
-    <child link="front_left_wheel_link" />
-  </joint>
-</robot>
+/home/nwhit210/omnicar_ws/src/omnicar/description/urdf/mecanum_wheel.urdf.xacro

File: install/omnicar/share/omnicar/description/urdf/mecanum_wheel_macro.xacro (robot description, xacro)
@@ -1,19 +1 @@
-<?xml version="1.0" ?>
-<robot name="mecanum_wheel" xmlns:xacro="http://ros.org/wiki/xacro">
-  <xacro:include filename="$(find omnicar)/description/urdf/wheel.xacro" />
-  <xacro:include filename="$(find omnicar)/description/urdf/rollers.xacro"  />
-  <xacro:macro name="mecanum_wheel" params="name side interface">
-    <xacro:wheel_link name="${name}" side="${side}" />
-    <xacro:rollers_link name="${name}" side="${side}" />
-    <transmission name="${name}_wheel_trans">
-      <type>transmission_interface/SimpleTransmission</type>
-      <joint name="${name}_wheel_joint">
-        <hardwareInterface>${interface}</hardwareInterface>
-      </joint>
-      <actuator name="${name}_wheel_motor">
-        <hardwareInterface>${interface}</hardwareInterface>
-        <mechanismReduction>1</mechanismReduction>
-      </actuator>
-    </transmission>
-  </xacro:macro>
-</robot>
+/home/nwhit210/omnicar_ws/src/omnicar/description/urdf/mecanum_wheel_macro.xacro

File: install/omnicar/share/omnicar/description/urdf/rollers.xacro (robot description, xacro)
@@ -1,63 +1 @@
-<?xml version="1.0" ?>
-<robot name="wheel" xmlns:xacro="http://www.ros.org/wiki/xacro">
-  <xacro:macro name="roller_origin" params="th side" >
-    <xacro:if value="${side==1}">
-      <origin xyz="0 ${0.0895*cos(th)} ${0.0895*sin(th)}" rpy="${atan(-tan(th)*sqrt(2.0))} ${asin(cos(th)/sqrt(2.0))} ${atan(sin(th))}"/>
-    </xacro:if>
-    <xacro:if value="${side==-1}">
-      <origin xyz="0 ${0.0895*cos(th)} ${0.0895*sin(th)}" rpy="${atan(-tan(th)*sqrt(2.0))} ${asin(-cos(th)/sqrt(2.0))} ${atan(-sin(th))}"/>
-    </xacro:if>
-  </xacro:macro>
-  <xacro:macro name="roller_loop" params="name side num loop" >
-    <xacro:if value="${loop}">
-      <link name="${name}_roller${loop}_link">
-        <visual>
-          <origin xyz="0 0 0" rpy="0 0 0" />
-          <geometry>
-            <mesh filename="$(find omnicar)/description/mesh/visual/roller.dae" scale="1 1 1" />
-          </geometry>
-        </visual>
-        <collision>
-          <geometry>
-            <mesh filename="$(find omnicar)/description/mesh/collision/roller.stl" scale="1 1 1" />
-          </geometry>
-        </collision>
-        <inertial>
-          <origin xyz="0 0 0" />
-          <mass value="0.3" />
-          <inertia ixx="0.00024000" ixy="0.0" ixz="0.0"
-                  iyy="0.00076000" iyz="0.0"
-                  izz="0.00076000" />
-        </inertial>
-      </link>
-      <joint name="${name}_roller${loop}_joint" type="continuous">
-        <xacro:roller_origin th="${radians(360/num*(loop-1))}" side="${side}"/>
-        <axis xyz="1 0 0"/>
-        <parent link="${name}_wheel_link" />
-        <child link="${name}_roller${loop}_link" />
-        <dynamics damping="0.001" friction="0.0001" />
-      </joint>
-      <transmission name="$${name}_roller${loop}_trans">
-        <type>transmission_interface/SimpleTransmission</type>
-        <joint name="${name}_roller${loop}_joint">
-          <hardwareInterface>hardware_interface/EffortJointInterface</hardwareInterface>
-        </joint>
-        <actuator name="${name}_roller${loop}_motor">
-          <hardwareInterface>hardware_interface/EffortJointInterface</hardwareInterface>
-          <mechanismReduction>1</mechanismReduction>
-        </actuator>
-      </transmission>
-      <gazebo reference="${name}_roller${loop}_link">
-        <mu1 value="0.8"/>
-        <mu2 value="0.8"/>
-        <kp value="10000000.0" />
-        <kd value="1.0" />
-        <fdir1 value="0 1 0"/>
-      </gazebo>
-      <xacro:roller_loop name="${name}" side="${side}" num="${num}" loop="${loop - 1}" />
-    </xacro:if>
-  </xacro:macro>
-  <xacro:macro name="rollers_link" params="name side">
-    <xacro:roller_loop name="${name}" side="${side}" num="15" loop="15" />
-  </xacro:macro>
-</robot>
+/home/nwhit210/omnicar_ws/src/omnicar/description/urdf/rollers.xacro

File: install/omnicar/share/omnicar/description/urdf/wheel.xacro (robot description, xacro)
@@ -1,32 +1 @@
-<?xml version="1.0" ?>
-<robot name="wheel" xmlns:xacro="http://www.ros.org/wiki/xacro">
-  <xacro:macro name="wheel_link" params="name side">
-    <link name="${name}_wheel_link">
-      <visual>
-        <origin xyz="0 0 0" rpy="0 0 0" />
-        <geometry>
-          <mesh filename="$(find omnicar)/description/mesh/visual/wheel.dae" scale="${side} 1 1" />
-        </geometry>
-      </visual>
-      <collision>
-        <geometry>
-          <mesh filename="$(find omnicar)/description/mesh/collision/wheel.stl" scale="${side} 1 1" />
-        </geometry>
-      </collision>
-      <inertial>
-        <origin xyz="0 0 0" />
-        <mass value="2.0" />
-        <inertia ixx="0.042025" ixy="0.0" ixz="0.0"
-                iyy="0.024279" iyz="0.0"
-                izz="0.024279" />
-      </inertial>
-    </link>
-    <gazebo reference="${name}_wheel_link">
-      <mu1 value="0.6"/>
-      <mu2 value="0.6"/>
-      <kp value="10000000.0" />
-      <kd value="1.0" />
-      <fdir1 value="0 1 0"/>
-    </gazebo>
-  </xacro:macro>
-</robot>
+/home/nwhit210/omnicar_ws/src/omnicar/description/urdf/wheel.xacro
