Commit message: First Working one!!

File: install/diffdrive_arduino/share/diffdrive_arduino/ros2_control/diffbot.ros2_control.xacro (robot description, xacro)
@@ -1,31 +1 @@
-<?xml version="1.0"?>
-<robot xmlns:xacro="http://www.ros.org/wiki/xacro">
-  <xacro:macro name="diffbot_ros2_control" params="name prefix">
-    <ros2_control name="${name}" type="system">
-      <hardware>
-        <plugin>diffdrive_arduino/DiffDriveArduinoHardware</plugin>
-        <param name="left_wheel_name">left_wheel_joint</param>
-        <param name="right_wheel_name">right_wheel_joint</param>
-        <param name="loop_rate">30</param>
-        <param name="device">/dev/serial/by-path/platform-fd500000.pcie-pci-0000:01:00.0-usb-0:1.3:1.0-port0</param>
-        <param name="baud_rate">57600</param>
-        <param name="timeout_ms">1000</param>
-        <param name="enc_counts_per_rev">3436</param>
-        <param name="pid_p">20</param>
-        <param name="pid_d">12</param>
-        <param name="pid_i">0</param>
-        <param name="pid_o">50</param>
-      </hardware>
-      <joint name="${prefix}left_wheel_joint">
-        <command_interface name="velocity"/>
-        <state_interface name="position"/>
-        <state_interface name="velocity"/>
-      </joint>
-      <joint name="${prefix}right_wheel_joint">
-        <command_interface name="velocity"/>
-        <state_interface name="position"/>
-        <state_interface name="velocity"/>
-      </joint>
-    </ros2_control>
-  </xacro:macro>
-</robot>
+/home/pi/omnicar_ws/src/diffdrive_arduino/description/ros2_control/diffbot.ros2_control.xacro

File: install/diffdrive_arduino/share/diffdrive_arduino/urdf/diffbot.materials.xacro (robot description, xacro)
@@ -1,31 +1 @@
-<?xml version="1.0"?>
-<!--
-Copied from ROS1 example:
-https://github.com/ros-simulation/gazebo_ros_demos/blob/kinetic-devel/rrbot_description/urdf/materials.xacro
--->
-<robot>
-  <material name="black">
-    <color rgba="0.0 0.0 0.0 1.0"/>
-  </material>
-  <material name="blue">
-    <color rgba="0.0 0.0 0.8 1.0"/>
-  </material>
-  <material name="green">
-    <color rgba="0.0 0.8 0.0 1.0"/>
-  </material>
-  <material name="grey">
-    <color rgba="0.2 0.2 0.2 1.0"/>
-  </material>
-  <material name="orange">
-    <color rgba="${255/255} ${108/255} ${10/255} 1.0"/>
-  </material>
-  <material name="brown">
-    <color rgba="${222/255} ${207/255} ${195/255} 1.0"/>
-  </material>
-  <material name="red">
-    <color rgba="0.8 0.0 0.0 1.0"/>
-  </material>
-  <material name="white">
-    <color rgba="1.0 1.0 1.0 1.0"/>
-  </material>
-</robot>
+/home/pi/omnicar_ws/src/diffdrive_arduino/description/urdf/diffbot.materials.xacro

File: install/diffdrive_arduino/share/diffdrive_arduino/urdf/diffbot.urdf.xacro (robot description, xacro)
@@ -1,13 +1 @@
-<?xml version="1.0"?>
-<!-- Basic differential drive mobile base -->
-<robot xmlns:xacro="http://www.ros.org/wiki/xacro" name="diffdrive_robot">
-  <xacro:arg name="prefix" default="" />
-  <xacro:include filename="$(find diffdrive_arduino)/urdf/diffbot_description.urdf.xacro" />
-  <!-- Import Rviz colors -->
-  <xacro:include filename="$(find diffdrive_arduino)/urdf/diffbot.materials.xacro" />
-  <!-- Import diffbot ros2_control description -->
-  <xacro:include filename="$(find diffdrive_arduino)/ros2_control/diffbot.ros2_control.xacro" />
-  <xacro:diffbot prefix="$(arg prefix)" />
-  <xacro:diffbot_ros2_control
-    name="DiffBot" prefix="$(arg prefix)" />
-</robot>
+/home/pi/omnicar_ws/src/diffdrive_arduino/description/urdf/diffbot.urdf.xacro

File: install/diffdrive_arduino/share/diffdrive_arduino/urdf/diffbot_description.urdf.xacro (robot description, xacro)
@@ -1,161 +1 @@
-<?xml version="1.0"?>
-<robot xmlns:xacro="http://www.ros.org/wiki/xacro">
-  <xacro:macro name="diffbot" params="prefix">
-  <!-- Constants for robot dimensions -->
-  <xacro:property name="PI" value="3.1415926535897931"/>
-  <xacro:property name="base_mass" value="0.3" /> <!-- arbitrary value for base mass -->
-  <xacro:property name="base_width" value="0.1" />
-  <xacro:property name="base_length" value="0.1" />
-  <xacro:property name="base_height" value="0.05" />
-  <xacro:property name="wheel_mass" value="0.3" /> <!-- arbitrary value for wheel mass -->
-  <xacro:property name="wheel_len" value="0.020" />
-  <xacro:property name="wheel_radius" value="0.015" />
-  <xacro:property name="caster_wheel_mass" value="0.1" /> <!-- arbitrary value for caster wheel mass -->
-  <xacro:property name="caster_wheel_radius" value="0.015" />
-  <xacro:property name="z_offset" value="-${base_height/2}" /> <!-- Space btw top of beam and the each joint -->
-  <!-- Base Link -->
-  <link name="${prefix}base_link">
-    <collision>
-      <origin xyz="0 0 0" rpy="0 0 0"/>
-      <geometry>
-        <box size="${base_width} ${base_length} ${base_height}"/>
-      </geometry>
-    </collision>
-    <visual>
-      <origin xyz="0 0 ${base_height/2}" rpy="0 0 0"/>
-      <geometry>
-        <box size="${base_width} ${base_length} ${base_height}"/>
-      </geometry>
-      <material name="orange"/>
-    </visual>
-    <inertial>
-      <origin xyz="0 0 0" rpy="0 0 0"/>
-      <mass value="${base_mass}"/>
-      <inertia
-        ixx="${base_mass / 12.0 * (base_length*base_length + base_height*base_height)}" ixy="0.0" ixz="0.0"
-        iyy="${base_mass / 12.0 * (base_height*base_height + base_width*base_width)}" iyz="0.0"
-        izz="${base_mass / 12.0 * (base_width*base_width + base_length*base_length)}"/>
-      </inertial>
-    </link>
-    <joint name="${prefix}left_wheel_joint" type="continuous">
-      <parent link="${prefix}base_link"/>
-      <child link="${prefix}left_wheel"/>
-      <origin xyz="0 -${base_width/2} ${z_offset}" rpy="0 0 0"/>
-      <axis xyz="0 1 0"/>
-      <dynamics damping="0.2"/>
-    </joint>
-    <!-- left wheel Link -->
-    <link name="${prefix}left_wheel">
-      <collision>
-        <origin xyz="0 0 0" rpy="${PI/2} 0 0"/>
-        <geometry>
-          <cylinder length="${wheel_len}" radius="${wheel_radius}"/>
-        </geometry>
-      </collision>
-      <visual>
-        <origin xyz="0 0 0" rpy="${PI/2} 0 0"/>
-        <geometry>
-          <cylinder length="${wheel_len}" radius="${wheel_radius}"/>
-        </geometry>
-        <material name="black"/>
-      </visual>
-      <inertial>
-        <origin xyz="0 0 0" rpy="${PI/2} 0 0"/>
-        <mass value="${wheel_mass}"/>
-        <inertia
-          ixx="${wheel_mass / 12.0 * (3*wheel_radius + wheel_len*wheel_len)}" ixy="0.0" ixz="0.0"
-          iyy="${wheel_mass / 12.0 * wheel_radius*wheel_radius}" iyz="0.0"
-          izz="${wheel_mass / 12.0 * wheel_radius*wheel_radius}"/>
-        </inertial>
-      </link>
-    <joint name="${prefix}right_wheel_joint" type="continuous">
-      <parent link="${prefix}base_link"/>
-      <child link="${prefix}right_wheel"/>
-      <origin xyz="0 ${base_width/2} ${z_offset}" rpy="0 0 0"/>
-      <axis xyz="0 1 0"/>
-      <dynamics damping="0.2"/>
-    </joint>
-    <!-- right wheel Link -->
-    <link name="${prefix}right_wheel">
-      <collision>
-        <origin xyz="0 0 0" rpy="${PI/2} 0 0"/>
-        <geometry>
-          <cylinder length="${wheel_len}" radius="${wheel_radius}"/>
-        </geometry>
-      </collision>
-      <visual>
-        <origin xyz="0 0 0" rpy="${PI/2} 0 0"/>
-        <geometry>
-          <cylinder length="${wheel_len}" radius="${wheel_radius}"/>
-        </geometry>
-        <material name="black"/>
-      </visual>
-      <inertial>
-        <origin xyz="0 0 0" rpy="${PI/2} 0 0"/>
-        <mass value="${wheel_mass}"/>
-        <inertia
-          ixx="${wheel_mass / 12.0 * (3*wheel_radius + wheel_len*wheel_len)}" ixy="0.0" ixz="0.0"
-          iyy="${wheel_mass / 12.0 * wheel_radius*wheel_radius}" iyz="0.0"
-          izz="${wheel_mass / 12.0 * wheel_radius*wheel_radius}"/>
-        </inertial>
-      </link>
-    <joint name="${prefix}caster_frontal_wheel_joint" type="fixed">
-      <parent link="${prefix}base_link"/>
-      <child link="${prefix}caster_frontal_wheel"/>
-      <origin xyz="${base_width/2 - caster_wheel_radius} 0 ${z_offset}" rpy="0 0 0"/>
-    </joint>
-    <!-- caster frontal wheel Link -->
-    <link name="${prefix}caster_frontal_wheel">
-      <collision>
-        <origin xyz="0 0 0" rpy="0 0 0"/>
-        <geometry>
-          <sphere radius="${caster_wheel_radius}"/>
-        </geometry>
-      </collision>
-      <visual>
-        <origin xyz="0 0 0" rpy="0 0 0"/>
-        <geometry>
-          <sphere radius="${caster_wheel_radius}"/>
-        </geometry>
-        <material name="white"/>
-      </visual>
-      <inertial>
-        <origin xyz="0 0 0" rpy="0 0 0"/>
-        <mass value="${caster_wheel_mass}"/>
-        <inertia
-          ixx="${caster_wheel_mass * 0.4 * (caster_wheel_radius * caster_wheel_radius)}" ixy="0.0" ixz="0.0"
-          iyy="${caster_wheel_mass * 0.4 * (caster_wheel_radius * caster_wheel_radius)}" iyz="0.0"
-          izz="${caster_wheel_mass * 0.4 * (caster_wheel_radius * caster_wheel_radius)}"/>
-        </inertial>
-      </link>
-    <joint name="${prefix}caster_rear_wheel_joint" type="fixed">
-      <parent link="${prefix}base_link"/>
-      <child link="${prefix}caster_rear_wheel"/>
-      <origin xyz="${-base_width/2 + caster_wheel_radius} 0 ${z_offset}" rpy="0 0 0"/>
-    </joint>
-    <!-- caster rear wheel Link -->
-    <link name="${prefix}caster_rear_wheel">
-      <collision>
-        <origin xyz="0 0 0" rpy="0 0 0"/>
-        <geometry>
-          <sphere radius="${caster_wheel_radius}"/>
-        </geometry>
-      </collision>
-      <visual>
-        <origin xyz="0 0 0" rpy="0 0 0"/>
-        <geometry>
-          <sphere radius="${caster_wheel_radius}"/>
-        </geometry>
-        <material name="white"/>
-      </visual>
-      <inertial>
-        <origin xyz="0 0 0" rpy="0 0 0"/>
-        <mass value="${caster_wheel_mass}"/>
-        <inertia
-          ixx="${caster_wheel_mass * 0.4 * (caster_wheel_radius * caster_wheel_radius)}" ixy="0.0" ixz="0.0"
-          iyy="${caster_wheel_mass * 0.4 * (caster_wheel_radius * caster_wheel_radius)}" iyz="0.0"
-          izz="${caster_wheel_mass * 0.4 * (caster_wheel_radius * caster_wheel_radius)}"/>
-        </inertial>
-      </link>
-  </xacro:macro>
-</robot>
+/home/pi/omnicar_ws/src/diffdrive_arduino/description/urdf/diffbot_description.urdf.xacro

File: install/omnicar/share/omnicar/description/camera.xacro (robot description, xacro)
@@ -1 +1 @@
-/home/nwhit210/omnicar_ws/src/omnicar/description/camera.xacro
+/home/pi/omnicar_ws/src/omnicar/description/camera.xacro

File: install/omnicar/share/omnicar/description/robot.urdf.xacro (robot description, xacro)
@@ -1 +1 @@
-/home/nwhit210/omnicar_ws/src/omnicar/description/robot.urdf.xacro
+/home/pi/omnicar_ws/src/omnicar/description/robot.urdf.xacro

File: install/omnicar/share/omnicar/description/robot_core.xacro (robot description, xacro)
@@ -1 +1 @@
-/home/nwhit210/omnicar_ws/src/omnicar/description/robot_core.xacro
+/home/pi/omnicar_ws/src/omnicar/description/robot_core.xacro

File: install/omnicar/share/omnicar/description/ros2_control.xacro (robot description, xacro)
@@ -1 +1 @@
-/home/nwhit210/omnicar_ws/src/omnicar/description/ros2_control.xacro
+/home/pi/omnicar_ws/src/omnicar/description/ros2_control.xacro

File: install/omnicar/share/omnicar/description/urdf/mecanum_wheel.urdf.xacro (robot description, xacro)
@@ -1 +1 @@
-/home/nwhit210/omnicar_ws/src/omnicar/description/urdf/mecanum_wheel.urdf.xacro
+/home/pi/omnicar_ws/src/omnicar/description/urdf/mecanum_wheel.urdf.xacro

File: install/omnicar/share/omnicar/description/urdf/mecanum_wheel_macro.xacro (robot description, xacro)
@@ -1 +1 @@
-/home/nwhit210/omnicar_ws/src/omnicar/description/urdf/mecanum_wheel_macro.xacro
+/home/pi/omnicar_ws/src/omnicar/description/urdf/mecanum_wheel_macro.xacro

File: install/omnicar/share/omnicar/description/urdf/rollers.xacro (robot description, xacro)
@@ -1 +1 @@
-/home/nwhit210/omnicar_ws/src/omnicar/description/urdf/rollers.xacro
+/home/pi/omnicar_ws/src/omnicar/description/urdf/rollers.xacro

File: install/omnicar/share/omnicar/description/urdf/wheel.xacro (robot description, xacro)
@@ -1 +1 @@
-/home/nwhit210/omnicar_ws/src/omnicar/description/urdf/wheel.xacro
+/home/pi/omnicar_ws/src/omnicar/description/urdf/wheel.xacro

File: install/ros2_control_demo_example_2/share/ros2_control_demo_example_2/ros2_control/diffbot.ros2_control.xacro (robot description, xacro)
@@ -1 +1,30 @@
-/home/nwhit210/omnicar_ws/src/example_2/description/ros2_control/diffbot.ros2_control.xacro
+<?xml version="1.0"?>
+<robot xmlns:xacro="http://www.ros.org/wiki/xacro">
+  <xacro:macro name="diffbot_ros2_control" params="name prefix use_mock_hardware">
+    <ros2_control name="${name}" type="system">
+      <xacro:unless value="${use_mock_hardware}">
+        <hardware>
+          <plugin>ros2_control_demo_example_2/DiffBotSystemHardware</plugin>
+          <param name="example_param_hw_start_duration_sec">0</param>
+          <param name="example_param_hw_stop_duration_sec">3.0</param>
+        </hardware>
+      </xacro:unless>
+      <xacro:if value="${use_mock_hardware}">
+        <hardware>
+          <plugin>mock_components/GenericSystem</plugin>
+          <param name="calculate_dynamics">true</param>
+        </hardware>
+      </xacro:if>
+      <joint name="${prefix}left_wheel_joint">
+        <command_interface name="velocity"/>
+        <state_interface name="position"/>
+        <state_interface name="velocity"/>
+      </joint>
+      <joint name="${prefix}right_wheel_joint">
+        <command_interface name="velocity"/>
+        <state_interface name="position"/>
+        <state_interface name="velocity"/>
+      </joint>
+    </ros2_control>
+  </xacro:macro>
+</robot>

File: install/ros2_control_demo_example_2/share/ros2_control_demo_example_2/urdf/diffbot.urdf.xacro (robot description, xacro)
@@ -1 +1,14 @@
-/home/nwhit210/omnicar_ws/src/example_2/description/urdf/diffbot.urdf.xacro
+<?xml version="1.0"?>
+<!-- Basic differential drive mobile base -->
+<robot xmlns:xacro="http://www.ros.org/wiki/xacro" name="diffdrive_robot">
+  <xacro:arg name="prefix" default="" />
+  <xacro:arg name="use_mock_hardware" default="false" />
+  <xacro:include filename="$(find ros2_control_demo_description)/diffbot/urdf/diffbot_description.urdf.xacro" />
+  <!-- Import Rviz colors -->
+  <xacro:include filename="$(find ros2_control_demo_description)/diffbot/urdf/diffbot.materials.xacro" />
+  <!-- Import diffbot ros2_control description -->
+  <xacro:include filename="$(find ros2_control_demo_example_2)/ros2_control/diffbot.ros2_control.xacro" />
+  <xacro:diffbot prefix="$(arg prefix)" />
+  <xacro:diffbot_ros2_control
+    name="DiffBot" prefix="$(arg prefix)" use_mock_hardware="$(arg use_mock_hardware)"/>
+</robot>

File: src/omnicar/description/ros2_control.xacro (robot description, xacro)
@@ -47,78 +47,50 @@
   </xacro:if>
   <xacro:unless value="$(arg sim_mode)">
-    <ros2_control name="RealBot" type="system">
-      <hardware>
-          <plugin>ros2_control_demo_example_2/DiffBotSystemHardware</plugin>
-          <param name="front_left_wheel_name">front_left_wheel_joint</param>
-          <param name="front_right_wheel_name">front_right_wheel_joint</param>
-          <param name="back_left_wheel_name">rear_left_wheel_joint</param>
-          <param name="back_right_wheel_name">rear_right_wheel_joint</param>
-          <param name="loop_rate">30.00</param>
-          <param name="device">/dev/ttyUSB0</param>
-          <param name="baud_rate">9600</param>
-          <param name="timeout_ms">1000</param>
+    <ros2_control name="RealRobot" type="system">
+        <hardware>
+            <plugin>diffdrive_arduino/DiffDriveArduinoHardware</plugin>
+            <param name="front_left_wheel_name">front_left_wheel_joint</param>
+            <param name="front_right_wheel_name">front_right_wheel_joint</param>
+            <param name="rear_left_wheel_name">rear_left_wheel_joint</param>
+            <param name="rear_right_wheel_name">rear_right_wheel_joint</param>
+            <param name="loop_rate">30</param>
+            <param name="device">/dev/ttyACM0</param>
+            <param name="baud_rate">57600</param>
+            <param name="timeout_ms">1000</param>
+            <param name="enc_counts_per_rev">3436</param>
         </hardware>
-      <joint name="rear_right_wheel_joint">
-          <command_interface name="velocity">
-              <param name="min">-10</param>
-              <param name="max">10</param>
-          </command_interface>
-          <state_interface name="position" />
-          <state_interface name="velocity" />
-      </joint>
-      <joint name="rear_left_wheel_joint">
-          <command_interface name="velocity">
-              <param name="min">-10</param>
-              <param name="max">10</param>
-          </command_interface>
-          <state_interface name="velocity" />
-          <state_interface name="position" />
-      </joint>
-      <joint name="front_right_wheel_joint">
-          <command_interface name="velocity">
-              <param name="min">-10</param>
-              <param name="max">10</param>
-          </command_interface>
-          <state_interface name="position" />
-          <state_interface name="velocity" />
-      </joint>
-      <joint name="front_left_wheel_joint">
-          <command_interface name="velocity">
-              <param name="min">-10</param>
-              <param name="max">10</param>
-          </command_interface>
-          <state_interface name="velocity" />
-          <state_interface name="position" />
-      </joint>
+        <joint name="rear_left_wheel_joint">
+            <command_interface name="velocity">
+                <param name="min">-10</param>
+                <param name="max">10</param>
+            </command_interface>
+            <state_interface name="position"/>
+            <state_interface name="velocity"/>
+        </joint>
+        <joint name="rear_right_wheel_joint">
+            <command_interface name="velocity">
+                <param name="min">-10</param>
+                <param name="max">10</param>
+            </command_interface>
+            <state_interface name="position"/>
+            <state_interface name="velocity"/>
+        </joint>
+        <joint name="front_left_wheel_joint">
+            <command_interface name="velocity">
+                <param name="min">-10</param>
+                <param name="max">10</param>
+            </command_interface>
+            <state_interface name="position"/>
+            <state_interface name="velocity"/>
+        </joint>
+        <joint name="front_right_wheel_joint">
+            <command_interface name="velocity">
+                <param name="min">-10</param>
+                <param name="max">10</param>
+            </command_interface>
+            <state_interface name="position"/>
+            <state_interface name="velocity"/>
+        </joint>
     </ros2_control>
-<!-- <ros2_control name="RealRobot" type="system">
-      <hardware>
-          <plugin>diffdrive_arduino/DiffDriveArduino</plugin>
-          <param name="left_wheel_name">back_left_wheel_joint</param>
-          <param name="right_wheel_name">back_right_wheel_joint</param>
-          <param name="loop_rate">30</param>
-          <param name="device">/dev/ttyUSB0</param>
-          <param name="baud_rate">57600</param>
-          <param name="timeout">1000</param>
-          <param name="enc_counts_per_rev">3436</param>
-      </hardware>
-      Note everything below here is the same as the Gazebo one
-      <joint name="back_left_wheel_joint">
-          <command_interface name="velocity">
-              <param name="min">-10</param>
-              <param name="max">10</param>
-          </command_interface>
-          <state_interface name="velocity"/>
-          <state_interface name="position"/>
-      </joint>
-      <joint name="back_right_wheel_joint">
-          <command_interface name="velocity">
-              <param name="min">-10</param>
-              <param name="max">10</param>
-          </command_interface>
-          <state_interface name="velocity"/>
-          <state_interface name="position"/>
-      </joint>
-    </ros2_control> -->
     <gazebo>
         <plugin name="gazebo_ros2_control" filename="libgazebo_ros2_control.so">
