Commit message: Latest update

File: install/diffdrive_arduino/share/diffdrive_arduino/ros2_control/diffbot.ros2_control.xacro (robot description, xacro)
@@ -1 +1,31 @@
-/home/pi/omnicar_ws/src/diffdrive_arduino/description/ros2_control/diffbot.ros2_control.xacro
+<?xml version="1.0"?>
+<robot xmlns:xacro="http://www.ros.org/wiki/xacro">
+  <xacro:macro name="diffbot_ros2_control" params="name prefix">
+    <ros2_control name="${name}" type="system">
+      <hardware>
+        <plugin>diffdrive_arduino/DiffDriveArduinoHardware</plugin>
+        <param name="left_wheel_name">left_wheel_joint</param>
+        <param name="right_wheel_name">right_wheel_joint</param>
+        <param name="loop_rate">30</param>
+        <param name="device">/dev/serial/by-path/platform-fd500000.pcie-pci-0000:01:00.0-usb-0:1.3:1.0-port0</param>
+        <param name="baud_rate">57600</param>
+        <param name="timeout_ms">1000</param>
+        <param name="enc_counts_per_rev">3436</param>
+        <param name="pid_p">20</param>
+        <param name="pid_d">12</param>
+        <param name="pid_i">0</param>
+        <param name="pid_o">50</param>
+      </hardware>
+      <joint name="${prefix}left_wheel_joint">
+        <command_interface name="velocity"/>
+        <state_interface name="position"/>
+        <state_interface name="velocity"/>
+      </joint>
+      <joint name="${prefix}right_wheel_joint">
+        <command_interface name="velocity"/>
+        <state_interface name="position"/>
+        <state_interface name="velocity"/>
+      </joint>
+    </ros2_control>
+  </xacro:macro>
+</robot>

File: install/diffdrive_arduino/share/diffdrive_arduino/urdf/diffbot.materials.xacro (robot description, xacro)
@@ -1 +1,31 @@
-/home/pi/omnicar_ws/src/diffdrive_arduino/description/urdf/diffbot.materials.xacro
+<?xml version="1.0"?>
+<!--
+Copied from ROS1 example:
+https://github.com/ros-simulation/gazebo_ros_demos/blob/kinetic-devel/rrbot_description/urdf/materials.xacro
+-->
+<robot>
+  <material name="black">
+    <color rgba="0.0 0.0 0.0 1.0"/>
+  </material>
+  <material name="blue">
+    <color rgba="0.0 0.0 0.8 1.0"/>
+  </material>
+  <material name="green">
+    <color rgba="0.0 0.8 0.0 1.0"/>
+  </material>
+  <material name="grey">
+    <color rgba="0.2 0.2 0.2 1.0"/>
+  </material>
+  <material name="orange">
+    <color rgba="${255/255} ${108/255} ${10/255} 1.0"/>
+  </material>
+  <material name="brown">
+    <color rgba="${222/255} ${207/255} ${195/255} 1.0"/>
+  </material>
+  <material name="red">
+    <color rgba="0.8 0.0 0.0 1.0"/>
+  </material>
+  <material name="white">
+    <color rgba="1.0 1.0 1.0 1.0"/>
+  </material>
+</robot>

File: install/diffdrive_arduino/share/diffdrive_arduino/urdf/diffbot.urdf.xacro (robot description, xacro)
@@ -1 +1,13 @@
-/home/pi/omnicar_ws/src/diffdrive_arduino/description/urdf/diffbot.urdf.xacro
+<?xml version="1.0"?>
+<!-- Basic differential drive mobile base -->
+<robot xmlns:xacro="http://www.ros.org/wiki/xacro" name="diffdrive_robot">
+  <xacro:arg name="prefix" default="" />
+  <xacro:include filename="$(find diffdrive_arduino)/urdf/diffbot_description.urdf.xacro" />
+  <!-- Import Rviz colors -->
+  <xacro:include filename="$(find diffdrive_arduino)/urdf/diffbot.materials.xacro" />
+  <!-- Import diffbot ros2_control description -->
+  <xacro:include filename="$(find diffdrive_arduino)/ros2_control/diffbot.ros2_control.xacro" />
+  <xacro:diffbot prefix="$(arg prefix)" />
+  <xacro:diffbot_ros2_control
+    name="DiffBot" prefix="$(arg prefix)" />
+</robot>

File: install/diffdrive_arduino/share/diffdrive_arduino/urdf/diffbot_description.urdf.xacro (robot description, xacro)
@@ -1 +1,161 @@
-/home/pi/omnicar_ws/src/diffdrive_arduino/description/urdf/diffbot_description.urdf.xacro
+<?xml version="1.0"?>
+<robot xmlns:xacro="http://www.ros.org/wiki/xacro">
+  <xacro:macro name="diffbot" params="prefix">
+  <!-- Constants for robot dimensions -->
+  <xacro:property name="PI" value="3.1415926535897931"/>
+  <xacro:property name="base_mass" value="0.3" /> <!-- arbitrary value for base mass -->
+  <xacro:property name="base_width" value="0.1" />
+  <xacro:property name="base_length" value="0.1" />
+  <xacro:property name="base_height" value="0.05" />
+  <xacro:property name="wheel_mass" value="0.3" /> <!-- arbitrary value for wheel mass -->
+  <xacro:property name="wheel_len" value="0.020" />
+  <xacro:property name="wheel_radius" value="0.015" />
+  <xacro:property name="caster_wheel_mass" value="0.1" /> <!-- arbitrary value for caster wheel mass -->
+  <xacro:property name="caster_wheel_radius" value="0.015" />
+  <xacro:property name="z_offset" value="-${base_height/2}" /> <!-- Space btw top of beam and the each joint -->
+  <!-- Base Link -->
+  <link name="${prefix}base_link">
+    <collision>
+      <origin xyz="0 0 0" rpy="0 0 0"/>
+      <geometry>
+        <box size="${base_width} ${base_length} ${base_height}"/>
+      </geometry>
+    </collision>
+    <visual>
+      <origin xyz="0 0 ${base_height/2}" rpy="0 0 0"/>
+      <geometry>
+        <box size="${base_width} ${base_length} ${base_height}"/>
+      </geometry>
+      <material name="orange"/>
+    </visual>
+    <inertial>
+      <origin xyz="0 0 0" rpy="0 0 0"/>
+      <mass value="${base_mass}"/>
+      <inertia
+        ixx="${base_mass / 12.0 * (base_length*base_length + base_height*base_height)}" ixy="0.0" ixz="0.0"
+        iyy="${base_mass / 12.0 * (base_height*base_height + base_width*base_width)}" iyz="0.0"
+        izz="${base_mass / 12.0 * (base_width*base_width + base_length*base_length)}"/>
+      </inertial>
+    </link>
+    <joint name="${prefix}left_wheel_joint" type="continuous">
+      <parent link="${prefix}base_link"/>
+      <child link="${prefix}left_wheel"/>
+      <origin xyz="0 -${base_width/2} ${z_offset}" rpy="0 0 0"/>
+      <axis xyz="0 1 0"/>
+      <dynamics damping="0.2"/>
+    </joint>
+    <!-- left wheel Link -->
+    <link name="${prefix}left_wheel">
+      <collision>
+        <origin xyz="0 0 0" rpy="${PI/2} 0 0"/>
+        <geometry>
+          <cylinder length="${wheel_len}" radius="${wheel_radius}"/>
+        </geometry>
+      </collision>
+      <visual>
+        <origin xyz="0 0 0" rpy="${PI/2} 0 0"/>
+        <geometry>
+          <cylinder length="${wheel_len}" radius="${wheel_radius}"/>
+        </geometry>
+        <material name="black"/>
+      </visual>
+      <inertial>
+        <origin xyz="0 0 0" rpy="${PI/2} 0 0"/>
+        <mass value="${wheel_mass}"/>
+        <inertia
+          ixx="${wheel_mass / 12.0 * (3*wheel_radius + wheel_len*wheel_len)}" ixy="0.0" ixz="0.0"
+          iyy="${wheel_mass / 12.0 * wheel_radius*wheel_radius}" iyz="0.0"
+          izz="${wheel_mass / 12.0 * wheel_radius*wheel_radius}"/>
+        </inertial>
+      </link>
+    <joint name="${prefix}right_wheel_joint" type="continuous">
+      <parent link="${prefix}base_link"/>
+      <child link="${prefix}right_wheel"/>
+      <origin xyz="0 ${base_width/2} ${z_offset}" rpy="0 0 0"/>
+      <axis xyz="0 1 0"/>
+      <dynamics damping="0.2"/>
+    </joint>
+    <!-- right wheel Link -->
+    <link name="${prefix}right_wheel">
+      <collision>
+        <origin xyz="0 0 0" rpy="${PI/2} 0 0"/>
+        <geometry>
+          <cylinder length="${wheel_len}" radius="${wheel_radius}"/>
+        </geometry>
+      </collision>
+      <visual>
+        <origin xyz="0 0 0" rpy="${PI/2} 0 0"/>
+        <geometry>
+          <cylinder length="${wheel_len}" radius="${wheel_radius}"/>
+        </geometry>
+        <material name="black"/>
+      </visual>
+      <inertial>
+        <origin xyz="0 0 0" rpy="${PI/2} 0 0"/>
+        <mass value="${wheel_mass}"/>
+        <inertia
+          ixx="${wheel_mass / 12.0 * (3*wheel_radius + wheel_len*wheel_len)}" ixy="0.0" ixz="0.0"
+          iyy="${wheel_mass / 12.0 * wheel_radius*wheel_radius}" iyz="0.0"
+          izz="${wheel_mass / 12.0 * wheel_radius*wheel_radius}"/>
+        </inertial>
+      </link>
+    <joint name="${prefix}caster_frontal_wheel_joint" type="fixed">
+      <parent link="${prefix}base_link"/>
+      <child link="${prefix}caster_frontal_wheel"/>
+      <origin xyz="${base_width/2 - caster_wheel_radius} 0 ${z_offset}" rpy="0 0 0"/>
+    </joint>
+    <!-- caster frontal wheel Link -->
+    <link name="${prefix}caster_frontal_wheel">
+      <collision>
+        <origin xyz="0 0 0" rpy="0 0 0"/>
+        <geometry>
+          <sphere radius="${caster_wheel_radius}"/>
+        </geometry>
+      </collision>
+      <visual>
+        <origin xyz="0 0 0" rpy="0 0 0"/>
+        <geometry>
+          <sphere radius="${caster_wheel_radius}"/>
+        </geometry>
+        <material name="white"/>
+      </visual>
+      <inertial>
+        <origin xyz="0 0 0" rpy="0 0 0"/>
+        <mass value="${caster_wheel_mass}"/>
+        <inertia
+          ixx="${caster_wheel_mass * 0.4 * (caster_wheel_radius * caster_wheel_radius)}" ixy="0.0" ixz="0.0"
+          iyy="${caster_wheel_mass * 0.4 * (caster_wheel_radius * caster_wheel_radius)}" iyz="0.0"
+          izz="${caster_wheel_mass * 0.4 * (caster_wheel_radius * caster_wheel_radius)}"/>
+        </inertial>
+      </link>
+    <joint name="${prefix}caster_rear_wheel_joint" type="fixed">
+      <parent link="${prefix}base_link"/>
+      <child link="${prefix}caster_rear_wheel"/>
+      <origin xyz="${-base_width/2 + caster_wheel_radius} 0 ${z_offset}" rpy="0 0 0"/>
+    </joint>
+    <!-- caster rear wheel Link -->
+    <link name="${prefix}caster_rear_wheel">
+      <collision>
+        <origin xyz="0 0 0" rpy="0 0 0"/>
+        <geometry>
+          <sphere radius="${caster_wheel_radius}"/>
+        </geometry>
+      </collision>
+      <visual>
+        <origin xyz="0 0 0" rpy="0 0 0"/>
+        <geometry>
+          <sphere radius="${caster_wheel_radius}"/>
+        </geometry>
+        <material name="white"/>
+      </visual>
+      <inertial>
+        <origin xyz="0 0 0" rpy="0 0 0"/>
+        <mass value="${caster_wheel_mass}"/>
+        <inertia
+          ixx="${caster_wheel_mass * 0.4 * (caster_wheel_radius * caster_wheel_radius)}" ixy="0.0" ixz="0.0"
+          iyy="${caster_wheel_mass * 0.4 * (caster_wheel_radius * caster_wheel_radius)}" iyz="0.0"
+          izz="${caster_wheel_mass * 0.4 * (caster_wheel_radius * caster_wheel_radius)}"/>
+        </inertial>
+      </link>
+  </xacro:macro>
+</robot>

File: install/omnicar/share/omnicar/description/camera.xacro (robot description, xacro)
@@ -1 +1,45 @@
-/home/pi/omnicar_ws/src/omnicar/description/camera.xacro
+<?xml version="1.0"?>
+<robot xmlns:xacro="http://www.ros.org/wiki/xacro">
+  <joint name="camera_joint" type="fixed">
+    <parent link="chassis"/>
+    <child link="camera_link"/>
+    <origin xyz="0.305 0 0.08" rpy="0 0 0"/>
+  </joint>
+  <link name="camera_link">
+    <visual>
+      <geometry>
+        <box size="0.010 0.03 0.03"/>
+      </geometry>
+      <material name="red"/>
+    </visual>
+  </link>
+  <gazebo reference="camera_link">
+    <material>Gazebo/Red</material>
+    <sensor name="camera" type="camera">
+      <pose> 0 0 0 0 0 0 </pose>
+      <visualize>true</visualize>
+      <update_rate>10</update_rate>
+      <camera>
+        <horizontal_fov>1.089</horizontal_fov>
+        <image>
+          <format>R8G8B8</format>
+          <width>640</width>
+          <height>480</height>
+        </image>
+        <clip>
+          <near>0.05</near>
+          <far>8.0</far>
+        </clip>
+      </camera>
+      <plugin name="camera_controller" filename="libgazebo_ros_camera.so">
+        <frame_name>camera_link_optical</frame_name>
+      </plugin>
+    </sensor>
+  </gazebo>
+  <joint name="camera_optical_joint" type="fixed">
+    <origin xyz="0 0 0" rpy="${-pi/2} 0 ${-pi/2}" />
+    <parent link="camera_link" />
+    <child link="camera_link_optical" />
+  </joint>
+  <link name="camera_link_optical"></link>
+</robot>

File: install/omnicar/share/omnicar/description/robot.urdf.xacro (robot description, xacro)
@@ -1 +1,7 @@
-/home/pi/omnicar_ws/src/omnicar/description/robot.urdf.xacro
+<?xml version="1.0"?>
+<robot xmlns:xacro="http://www.ros.org/wiki/xacro"  name="robot">
+  <xacro:arg name='sim_mode' default='true'/>
+    <xacro:include filename="robot_core.xacro" />
+    <xacro:include filename="ros2_control.xacro" />
+    <!-- <xacro:include filename="camera.xacro" /> add camera -->
+</robot>

File: install/omnicar/share/omnicar/description/robot_core.xacro (robot description, xacro)
@@ -1 +1,58 @@
-/home/pi/omnicar_ws/src/omnicar/description/robot_core.xacro
+<?xml version="1.0" ?>
+<robot name="mecanum_wheel_robot" xmlns:xacro="http://ros.org/wiki/xacro">
+  <xacro:include filename="$(find omnicar)/description/urdf/mecanum_wheel_macro.xacro" />
+  <link name="base_link">
+    <visual>
+      <geometry>
+        <box size="0.7 0.4 0.3" />
+      </geometry>
+    </visual>
+    <collision>
+      <geometry>
+        <box size="0.7 0.4 0.3" />
+      </geometry>
+    </collision>
+    <inertial>
+      <origin xyz="0 0 0" />
+      <mass value="10.0" />
+      <inertia ixx="0.83333" ixy="0.0" ixz="0.0"
+              iyy="1.9333" iyz="0.0"
+              izz="2.1667" />
+    </inertial>
+  </link>
+  <gazebo reference="base_link">
+    <mu1 value="0.6"/>
+    <mu2 value="0.6"/>
+    <kp value="10000000.0" />
+    <kd value="1.0" />
+    <fdir1 value="0 1 0"/>
+  </gazebo>
+  <xacro:mecanum_wheel name="front_right" side="1"  interface="hardware_interface/EffortJointInterface"/>
+  <xacro:mecanum_wheel name="front_left"  side="-1" interface="hardware_interface/EffortJointInterface"/>
+  <xacro:mecanum_wheel name="rear_right"  side="-1" interface="hardware_interface/EffortJointInterface"/>
+  <xacro:mecanum_wheel name="rear_left"   side="1"  interface="hardware_interface/EffortJointInterface"/>
+  <joint name="front_right_wheel_joint" type="continuous">
+    <origin xyz="0.3 -0.25 -0.1" rpy="0 0 ${pi/2}" />
+    <axis xyz="1 0 0" />
+    <parent link="base_link" />
+    <child link="front_right_wheel_link" />
+  </joint>
+  <joint name="front_left_wheel_joint" type="continuous">
+    <origin xyz="0.3 0.25 -0.1" rpy="0 0 ${pi/2}" />
+    <axis xyz="1 0 0" />
+    <parent link="base_link" />
+    <child link="front_left_wheel_link" />
+  </joint>
+  <joint name="rear_right_wheel_joint" type="continuous">
+    <origin xyz="-0.3 -0.25 -0.1" rpy="0 0 ${pi/2}" />
+    <axis xyz="1 0 0" />
+    <parent link="base_link" />
+    <child link="rear_right_wheel_link" />
+  </joint>
+  <joint name="rear_left_wheel_joint" type="continuous">
+    <origin xyz="-0.3 0.25 -0.1" rpy="0 0 ${pi/2}" />
+    <axis xyz="1 0 0" />
+    <parent link="base_link" />
+    <child link="rear_left_wheel_link" />
+  </joint>
+</robot>

File: install/omnicar/share/omnicar/description/ros2_control.xacro (robot description, xacro)
@@ -1 +1,101 @@
-/home/pi/omnicar_ws/src/omnicar/description/ros2_control.xacro
+<?xml version="1.0"?>
+<robot xmlns:xacro="http://www.ros.org/wiki/xacro">
+  <xacro:if value="$(arg sim_mode)">
+    <ros2_control name="GazeboSystem" type="system">
+      <hardware>
+          <plugin>gazebo_ros2_control/GazeboSystem</plugin>
+      </hardware>
+      <joint name="rear_right_wheel_joint">
+          <command_interface name="velocity">
+              <param name="min">-10</param>
+              <param name="max">10</param>
+          </command_interface>
+          <state_interface name="position" />
+          <state_interface name="velocity" />
+      </joint>
+      <joint name="rear_left_wheel_joint">
+          <command_interface name="velocity">
+              <param name="min">-10</param>
+              <param name="max">10</param>
+          </command_interface>
+          <state_interface name="velocity" />
+          <state_interface name="position" />
+      </joint>
+      <joint name="front_right_wheel_joint">
+          <command_interface name="velocity">
+              <param name="min">-10</param>
+              <param name="max">10</param>
+          </command_interface>
+          <state_interface name="position" />
+          <state_interface name="velocity" />
+      </joint>
+      <joint name="front_left_wheel_joint">
+          <command_interface name="velocity">
+              <param name="min">-10</param>
+              <param name="max">10</param>
+          </command_interface>
+          <state_interface name="velocity" />
+          <state_interface name="position" />
+      </joint>
+    </ros2_control>
+    <gazebo>
+      <plugin name="gazebo_ros2_control" filename="libgazebo_ros2_control.so">
+        <parameters>$(find omnicar)/config/my_controllers.yaml</parameters>
+        <parameters>$(find omnicar)/config/sim.yaml</parameters>
+      </plugin>
+    </gazebo>
+  </xacro:if>
+  <xacro:unless value="$(arg sim_mode)">
+    <ros2_control name="RealRobot" type="system">
+        <hardware>
+            <plugin>diffdrive_arduino/DiffDriveArduinoHardware</plugin>
+            <param name="front_left_wheel_name">front_left_wheel_joint</param>
+            <param name="front_right_wheel_name">front_right_wheel_joint</param>
+            <param name="rear_left_wheel_name">rear_left_wheel_joint</param>
+            <param name="rear_right_wheel_name">rear_right_wheel_joint</param>
+            <param name="loop_rate">30</param>
+            <param name="device">/dev/ttyACM0</param>
+            <param name="baud_rate">57600</param>
+            <param name="timeout_ms">1000</param>
+            <param name="enc_counts_per_rev">3436</param>
+        </hardware>
+        <joint name="rear_left_wheel_joint">
+            <command_interface name="velocity">
+                <param name="min">-10</param>
+                <param name="max">10</param>
+            </command_interface>
+            <state_interface name="position"/>
+            <state_interface name="velocity"/>
+        </joint>
+        <joint name="rear_right_wheel_joint">
+            <command_interface name="velocity">
+                <param name="min">-10</param>
+                <param name="max">10</param>
+            </command_interface>
+            <state_interface name="position"/>
+            <state_interface name="velocity"/>
+        </joint>
+        <joint name="front_left_wheel_joint">
+            <command_interface name="velocity">
+                <param name="min">-10</param>
+                <param name="max">10</param>
+            </command_interface>
+            <state_interface name="position"/>
+            <state_interface name="velocity"/>
+        </joint>
+        <joint name="front_right_wheel_joint">
+            <command_interface name="velocity">
+                <param name="min">-10</param>
+                <param name="max">10</param>
+            </command_interface>
+            <state_interface name="position"/>
+            <state_interface name="velocity"/>
+        </joint>
+    </ros2_control>
+    <gazebo>
+        <plugin name="gazebo_ros2_control" filename="libgazebo_ros2_control.so">
+          <parameters>$(find omnicar)/config/my_controllers.yaml</parameters>
+        </plugin>
+    </gazebo>
+  </xacro:unless>
+</robot>

File: install/omnicar/share/omnicar/description/urdf/mecanum_wheel.urdf.xacro (robot description, xacro)
@@ -1 +1,19 @@
-/home/pi/omnicar_ws/src/omnicar/description/urdf/mecanum_wheel.urdf.xacro
+<?xml version="1.0" ?>
+<robot name="mecanum_wheel_robot" xmlns:xacro="http://ros.org/wiki/xacro">
+  <xacro:include filename="$(find omnicar)/description/urdf/mecanum_wheel_macro.xacro" />
+  <xacro:mecanum_wheel name="front_right" side="1" interface="hardware_interface/EffortJointInterface" />
+  <xacro:mecanum_wheel name="front_left" side="-1" interface="hardware_interface/EffortJointInterface" />
+  <link name="map">
+    <origin xyz="0 0 0" rpy="0 0 0" />
+  </link>
+  <joint name="virtual_map_right" type="fixed">
+    <origin xyz="0.1 0.2 0" />
+    <parent link="map" />
+    <child link="front_right_wheel_link" />
+  </joint>
+  <joint name="virtual_map_left" type="fixed">
+    <origin xyz="-0.1 0.2 0" />
+    <parent link="map" />
+    <child link="front_left_wheel_link" />
+  </joint>
+</robot>

File: install/omnicar/share/omnicar/description/urdf/mecanum_wheel_macro.xacro (robot description, xacro)
@@ -1 +1,19 @@
-/home/pi/omnicar_ws/src/omnicar/description/urdf/mecanum_wheel_macro.xacro
+<?xml version="1.0" ?>
+<robot name="mecanum_wheel" xmlns:xacro="http://ros.org/wiki/xacro">
+  <xacro:include filename="$(find omnicar)/description/urdf/wheel.xacro" />
+  <xacro:include filename="$(find omnicar)/description/urdf/rollers.xacro"  />
+  <xacro:macro name="mecanum_wheel" params="name side interface">
+    <xacro:wheel_link name="${name}" side="${side}" />
+    <xacro:rollers_link name="${name}" side="${side}" />
+    <transmission name="${name}_wheel_trans">
+      <type>transmission_interface/SimpleTransmission</type>
+      <joint name="${name}_wheel_joint">
+        <hardwareInterface>${interface}</hardwareInterface>
+      </joint>
+      <actuator name="${name}_wheel_motor">
+        <hardwareInterface>${interface}</hardwareInterface>
+        <mechanismReduction>1</mechanismReduction>
+      </actuator>
+    </transmission>
+  </xacro:macro>
+</robot>
