Commit message: Latest update

File: install/omnicar/share/omnicar/description/urdf/rollers.xacro (robot description, xacro)
@@ -1 +1,63 @@
-/home/pi/omnicar_ws/src/omnicar/description/urdf/rollers.xacro
+<?xml version="1.0" ?>
+<robot name="wheel" xmlns:xacro="http://www.ros.org/wiki/xacro">
+  <xacro:macro name="roller_origin" params="th side" >
+    <xacro:if value="${side==1}">
+      <origin xyz="0 ${0.0895*cos(th)} ${0.0895*sin(th)}" rpy="${atan(-tan(th)*sqrt(2.0))} ${asin(cos(th)/sqrt(2.0))} ${atan(sin(th))}"/>
+    </xacro:if>
+    <xacro:if value="${side==-1}">
+      <origin xyz="0 ${0.0895*cos(th)} ${0.0895*sin(th)}" rpy="${atan(-tan(th)*sqrt(2.0))} ${asin(-cos(th)/sqrt(2.0))} ${atan(-sin(th))}"/>
+    </xacro:if>
+  </xacro:macro>
+  <xacro:macro name="roller_loop" params="name side num loop" >
+    <xacro:if value="${loop}">
+      <link name="${name}_roller${loop}_link">
+        <visual>
+          <origin xyz="0 0 0" rpy="0 0 0" />
+          <geometry>
+            <mesh filename="$(find omnicar)/description/mesh/visual/roller.dae" scale="1 1 1" />
+          </geometry>
+        </visual>
+        <collision>
+          <geometry>
+            <mesh filename="$(find omnicar)/description/mesh/collision/roller.stl" scale="1 1 1" />
+          </geometry>
+        </collision>
+        <inertial>
+          <origin xyz="0 0 0" />
+          <mass value="0.3" />
+          <inertia ixx="0.00024000" ixy="0.0" ixz="0.0"
+                  iyy="0.00076000" iyz="0.0"
+                  izz="0.00076000" />
+        </inertial>
+      </link>
+      <joint name="${name}_roller${loop}_joint" type="continuous">
+        <xacro:roller_origin th="${radians(360/num*(loop-1))}" side="${side}"/>
+        <axis xyz="1 0 0"/>
+        <parent link="${name}_wheel_link" />
+        <child link="${name}_roller${loop}_link" />
+        <dynamics damping="0.001" friction="0.0001" />
+      </joint>
+      <transmission name="$${name}_roller${loop}_trans">
+        <type>transmission_interface/SimpleTransmission</type>
+        <joint name="${name}_roller${loop}_joint">
+          <hardwareInterface>hardware_interface/EffortJointInterface</hardwareInterface>
+        </joint>
+        <actuator name="${name}_roller${loop}_motor">
+          <hardwareInterface>hardware_interface/EffortJointInterface</hardwareInterface>
+          <mechanismReduction>1</mechanismReduction>
+        </actuator>
+      </transmission>
+      <gazebo reference="${name}_roller${loop}_link">
+        <mu1 value="0.8"/>
+        <mu2 value="0.8"/>
+        <kp value="10000000.0" />
+        <kd value="1.0" />
+        <fdir1 value="0 1 0"/>
+      </gazebo>
+      <xacro:roller_loop name="${name}" side="${side}" num="${num}" loop="${loop - 1}" />
+    </xacro:if>
+  </xacro:macro>
+  <xacro:macro name="rollers_link" params="name side">
+    <xacro:roller_loop name="${name}" side="${side}" num="15" loop="15" />
+  </xacro:macro>
+</robot>

File: install/omnicar/share/omnicar/description/urdf/wheel.xacro (robot description, xacro)
@@ -1 +1,32 @@
-/home/pi/omnicar_ws/src/omnicar/description/urdf/wheel.xacro
+<?xml version="1.0" ?>
+<robot name="wheel" xmlns:xacro="http://www.ros.org/wiki/xacro">
+  <xacro:macro name="wheel_link" params="name side">
+    <link name="${name}_wheel_link">
+      <visual>
+        <origin xyz="0 0 0" rpy="0 0 0" />
+        <geometry>
+          <mesh filename="$(find omnicar)/description/mesh/visual/wheel.dae" scale="${side} 1 1" />
+        </geometry>
+      </visual>
+      <collision>
+        <geometry>
+          <mesh filename="$(find omnicar)/description/mesh/collision/wheel.stl" scale="${side} 1 1" />
+        </geometry>
+      </collision>
+      <inertial>
+        <origin xyz="0 0 0" />
+        <mass value="2.0" />
+        <inertia ixx="0.042025" ixy="0.0" ixz="0.0"
+                iyy="0.024279" iyz="0.0"
+                izz="0.024279" />
+      </inertial>
+    </link>
+    <gazebo reference="${name}_wheel_link">
+      <mu1 value="0.6"/>
+      <mu2 value="0.6"/>
+      <kp value="10000000.0" />
+      <kd value="1.0" />
+      <fdir1 value="0 1 0"/>
+    </gazebo>
+  </xacro:macro>
+</robot>
